File: superduro.sch (KiCad schematic (older format))
At the start: 10 parts, among them Q1 BS170

Commit message: added in/out/pwr jacks
Parts:
- added J1: Input, jacks:2PADS_TS, symbol Connector:AudioJack2
- added J2: Output, jacks:2PADS_TS, symbol Connector:AudioJack2
- added J3: Power, jacks:DC_TS, symbol Connector:Barrel_Jack
- C1: footprint (none) -> caps-film:0.2_22.MED
- C2: footprint (none) -> caps-elec:0502
- D1, D2: footprint (none) -> diodes:DO35-2
- Q1: footprint Package_TO_SOT_THT:TO-92_Inline -> transistors-BJT:TO92
- R1, R2, R3, R4: footprint (none) -> resistors:0.3%22.B
- RV1: footprint (none) -> potentiometers:16MM_C.MOUNT
Connections:
- wire segments 27 -> 35
Changed lines of the file:
@@
 Connection ~ 2350 2400
 Wire Wire Line
+	1400 3000 1750 3000
+Wire Wire Line
+	1400 3100 1500 3100
+Wire Wire Line
 	1450 950  2350 950
 Wire Wire Line
 	1500 1850 1800 1850
 Wire Wire Line
+	1750 3000 1750 3100
+Wire Wire Line
 	2100 1850 2350 1850
 Wire Wire Line
@@
 	2350 2400 2350 2450
 Wire Wire Line
+	2700 3000 3150 3000
+Wire Wire Line
+	2700 3100 2850 3100
+Wire Wire Line
 	2950 1450 3600 1450
 Wire Wire Line
@@
 	2950 2300 2950 2450
 Wire Wire Line
+	3150 3000 3150 3100
+Wire Wire Line
 	3300 1850 3300 1650
 Wire Wire Line
@@
 Wire Wire Line
 	3600 2400 3600 2450
+Wire Wire Line
+	4050 2950 4150 2950
+Wire Wire Line
+	4050 3150 4150 3150
 Wire Wire Line
 	4300 1450 4300 1850
@@
 Text GLabel 1500 1850 0    50   Input ~ 0
 IN
+Text GLabel 1500 3100 2    50   Input ~ 0
+IN
+Text GLabel 2850 3100 2    50   Output ~ 0
+OUT
 Text GLabel 4800 1850 2    50   Output ~ 0
 OUT
@@
 $EndComp
 $Comp
+L power:+9V #PWR08
+U 1 1 00000000
+P 4150 2950
+F 0 "#PWR08" H 4150 2800 50  0001 C CNN
+F 1 "+9V" V 4165 3078 50  0000 L CNN
+F 2 "" H 4150 2950 50  0001 C CNN
+F 3 "" H 4150 2950 50  0001 C CNN
+	1    4150 2950
+	0    1    1    0
+$EndComp
+$Comp
+L power:GND #PWR06
+U 1 1 00000000
+P 1750 3100
+F 0 "#PWR06" H 1750 2850 50  0001 C CNN
+F 1 "GND" H 1755 2927 50  0000 C CNN
+F 2 "" H 1750 3100 50  0001 C CNN
+F 3 "" H 1750 3100 50  0001 C CNN
+	1    1750 3100
+	1    0    0    -1
+$EndComp
+$Comp
 L power:GND #PWR02
 U 1 1 00000000
@@
 $EndComp
 $Comp
+L power:GND #PWR07
+U 1 1 00000000
+P 3150 3100
+F 0 "#PWR07" H 3150 2850 50  0001 C CNN
+F 1 "GND" H 3155 2927 50  0000 C CNN
+F 2 "" H 3150 3100 50  0001 C CNN
+F 3 "" H 3150 3100 50  0001 C CNN
+	1    3150 3100
+	1    0    0    -1
+$EndComp
+$Comp
 L power:GND #PWR04
 U 1 1 00000000
@@
 $EndComp
 $Comp
+L power:GND #PWR09
+U 1 1 00000000
+P 4150 3150
+F 0 "#PWR09" H 4150 2900 50  0001 C CNN
+F 1 "GND" H 4155 2977 50  0000 C CNN
+F 2 "" H 4150 3150 50  0001 C CNN
+F 3 "" H 4150 3150 50  0001 C CNN
+	1    4150 3150
+	1    0    0    -1
+$EndComp
+$Comp
 L power:GND #PWR05
 U 1 1 00000000
@@
 F 0 "R2" H 3020 1645 50  0000 L CNN
 F 1 "10M" H 3020 1555 50  0000 L CNN
-F 2 "" V 2880 1600 50  0001 C CNN
+F 2 "resistors:0.3%22.B" V 2880 1600 50  0001 C CNN
 F 3 "~" H 2950 1600 50  0001 C CNN
 	1    2950 1600
@@
 F 0 "R1" H 3020 2195 50  0000 L CNN
 F 1 "10M" H 3020 2105 50  0000 L CNN
-F 2 "" V 2880 2150 50  0001 C CNN
+F 2 "resistors:0.3%22.B" V 2880 2150 50  0001 C CNN
 F 3 "~" H 2950 2150 50  0001 C CNN
 	1    2950 2150
@@
 F 0 "R3" H 3670 1145 50  0000 L CNN
 F 1 "5k1" H 3670 1055 50  0000 L CNN
-F 2 "" V 3530 1100 50  0001 C CNN
+F 2 "resistors:0.3%22.B" V 3530 1100 50  0001 C CNN
 F 3 "~" H 3600 1100 50  0001 C CNN
 	1    3600 1100
@@
 F 0 "R4" H 4370 2195 50  0000 L CNN
 F 1 "100k" H 4370 2105 50  0000 L CNN
-F 2 "" V 4230 2150 50  0001 C CNN
+F 2 "resistors:0.3%22.B" V 4230 2150 50  0001 C CNN
 F 3 "~" H 4300 2150 50  0001 C CNN
 	1    4300 2150
@@
 F 0 "D1" V 2305 1679 50  0000 L CNN
 F 1 "1N4148" V 2395 1679 50  0000 L CNN
-F 2 "" H 2350 1600 50  0001 C CNN
+F 2 "diodes:DO35-2" H 2350 1600 50  0001 C CNN
 F 3 "~" H 2350 1600 50  0001 C CNN
 	1    2350 1600
@@
 F 0 "D2" V 2305 2229 50  0000 L CNN
 F 1 "1N4148" V 2395 2229 50  0000 L CNN
-F 2 "" H 2350 2150 50  0001 C CNN
+F 2 "diodes:DO35-2" H 2350 2150 50  0001 C CNN
 F 3 "~" H 2350 2150 50  0001 C CNN
 	1    2350 2150
@@
 F 0 "C1" V 2201 1850 50  0000 C CNN
 F 1 "100n" V 2110 1850 50  0000 C CNN
-F 2 "" H 1988 1700 50  0001 C CNN
+F 2 "caps-film:0.2_22.MED" H 1988 1700 50  0001 C CNN
 F 3 "~" H 1950 1850 50  0001 C CNN
 	1    1950 1850
@@
 F 0 "C2" V 4404 1450 50  0000 C CNN
 F 1 "10u" V 4313 1450 50  0000 C CNN
-F 2 "" H 4188 1300 50  0001 C CNN
+F 2 "caps-elec:0502" H 4188 1300 50  0001 C CNN
 F 3 "~" H 4150 1450 50  0001 C CNN
 	1    4150 1450
@@
 F 0 "RV1" H 3530 2105 50  0000 R CNN
 F 1 "C5k" H 3530 2195 50  0000 R CNN
-F 2 "" H 3600 2150 50  0001 C CNN
+F 2 "potentiometers:16MM_C.MOUNT" H 3600 2150 50  0001 C CNN
 F 3 "~" H 3600 2150 50  0001 C CNN
 	1    3600 2150
@@
 $EndComp
 $Comp
+L Connector:AudioJack2 J1
+U 1 1 00000000
+P 1200 3100
+F 0 "J1" H 1232 3423 50  0000 C CNN
+F 1 "Input" H 1232 3332 50  0000 C CNN
+F 2 "jacks:2PADS_TS" H 1200 3100 50  0001 C CNN
+F 3 "~" H 1200 3100 50  0001 C CNN
+	1    1200 3100
+	1    0    0    -1
+$EndComp
+$Comp
+L Connector:AudioJack2 J2
+U 1 1 00000000
+P 2500 3100
+F 0 "J2" H 2532 3423 50  0000 C CNN
+F 1 "Output" H 2532 3332 50  0000 C CNN
+F 2 "jacks:2PADS_TS" H 2500 3100 50  0001 C CNN
+F 3 "~" H 2500 3100 50  0001 C CNN
+	1    2500 3100
+	1    0    0    -1
+$EndComp
+$Comp
+L Connector:Barrel_Jack J3
+U 1 1 00000000
+P 3750 3050
+F 0 "J3" H 3520 3008 50  0000 R CNN
+F 1 "Power" H 3520 3099 50  0000 R CNN
+F 2 "jacks:DC_TS" H 3800 3010 50  0001 C CNN
+F 3 "~" H 3800 3010 50  0001 C CNN
+	1    3750 3050
+	1    0    0    1
+$EndComp
+$Comp
 L Transistor_FET:BS170 Q1
 U 1 1 00000000
@@
 F 0 "Q1" H 3705 1695 50  0000 L CNN
 F 1 "BS170" H 3705 1605 50  0000 L CNN
-F 2 "Package_TO_SOT_THT:TO-92_Inline" H 3700 1575 50  0001 L CIN
+F 2 "transistors-BJT:TO92" H 3700 1575 50  0001 L CIN
 F 3 "http://www.fairchildsemi.com/ds/BS/BS170.pdf" H 3500 1650 50  0001 L CNN
 	1    3500 1650

Commit message: v0.1: initial version
Parts:
- removed J1: Input, jacks:2PADS_TS, symbol Connector:AudioJack2
- removed J2: Output, jacks:2PADS_TS, symbol Connector:AudioJack2
- removed J3: Power, jacks:DC_TS, symbol Connector:Barrel_Jack
- added D3: LED, LED_THT:LED_D3.0mm, symbol Device:LED
- added J1: Stomp_Connector, rockola_kicad_footprints:Stomp_4pin, symbol rockola_kicad_symbols:Stomp_Connector
- added J2: Conn_01x02, rockola_kicad_footprints:Power_Header_2pin_VERTICAL, symbol Connector_Generic:Conn_01x02
- added J3: Conn_01x01, rockola_kicad_footprints:V+_TOP_TEXT, symbol Connector_Generic:Conn_01x01
- added J4: Conn_01x01, supply_pins:PAD1, symbol Connector_Generic:Conn_01x01
- added R5: 4k7, resistors:0.3%22.B, symbol Device:R
- Q1: footprint transistors-BJT:TO92 -> rockola_kicad_footprints:TO92_DGS
- RV1: footprint potentiometers:16MM_C.MOUNT -> rockola_kicad_footprints:16mm_BoardMount
Connections:
- net labels added: LED-
- wire segments 35 -> 37
Changed lines of the file:
@@
 EESchema Schematic File Version 5
-EELAYER 31 0
+EELAYER 32 0
 EELAYER END
 $Descr A4 11693 8268
@@
 $EndDescr
 Connection ~ 4300 1850
-Connection ~ 2350 1850
+Connection ~ 2350 950
 Connection ~ 3600 1450
-Connection ~ 2350 950
+Connection ~ 1450 950
 Connection ~ 3600 2400
-Connection ~ 1450 950
 Connection ~ 2950 1850
 Connection ~ 2350 2400
-Wire Wire Line
-	1400 3000 1750 3000
-Wire Wire Line
-	1400 3100 1500 3100
+Connection ~ 2350 1850
+Wire Wire Line
+	1150 2850 1300 2850
 Wire Wire Line
 	1450 950  2350 950
@@
 	1500 1850 1800 1850
 Wire Wire Line
-	1750 3000 1750 3100
+	1600 2850 1650 2850
+Wire Wire Line
+	1950 2700 1950 2850
+Wire Wire Line
+	2050 3000 2050 3100
+Wire Wire Line
+	2050 3000 2500 3000
 Wire Wire Line
 	2100 1850 2350 1850
@@
 	2350 2400 2350 2450
 Wire Wire Line
-	2700 3000 3150 3000
-Wire Wire Line
-	2700 3100 2850 3100
+	2350 2900 2500 2900
+Wire Wire Line
+	2350 3100 2500 3100
+Wire Wire Line
+	2350 3200 2500 3200
 Wire Wire Line
 	2950 1450 3600 1450
@@
 	2950 2300 2950 2450
 Wire Wire Line
-	3150 3000 3150 3100
-Wire Wire Line
 	3300 1850 3300 1650
 Wire Wire Line
@@
 	3600 2400 3600 2450
 Wire Wire Line
-	4050 2950 4150 2950
-Wire Wire Line
-	4050 3150 4150 3150
+	3750 2950 3900 2950
+Wire Wire Line
+	3750 3050 3900 3050
 Wire Wire Line
 	4300 1450 4300 1850
@@
 Wire Wire Line
 	4300 2300 4300 2450
+Text GLabel 1150 2850 0    50   Input ~ 0
+LED-
 Text GLabel 1500 1850 0    50   Input ~ 0
 IN
-Text GLabel 1500 3100 2    50   Input ~ 0
+Text GLabel 2350 2900 0    50   Input ~ 0
 IN
-Text GLabel 2850 3100 2    50   Output ~ 0
+Text GLabel 2350 3100 0    50   Input ~ 0
+LED-
+Text GLabel 2350 3200 0    50   Output ~ 0
 OUT
 Text GLabel 4800 1850 2    50   Output ~ 0
@@
 $Comp
 L power:PWR_FLAG #FLG01
-U 1 1 00000000
+U 1 1 5E75D056
 P 1450 950
 F 0 "#FLG01" H 1450 1025 50  0001 C CNN
@@
 $Comp
 L power:PWR_FLAG #FLG02
-U 1 1 00000000
+U 1 1 5E75D069
 P 2350 2400
 F 0 "#FLG02" H 2350 2475 50  0001 C CNN
@@
 $Comp
 L power:+9V #PWR01
-U 1 1 00000000
+U 1 1 5E75D075
 P 1450 950
 F 0 "#PWR01" H 1450 800 50  0001 C CNN
@@
 $EndComp
 $Comp
-L power:+9V #PWR08
-U 1 1 00000000
-P 4150 2950
-F 0 "#PWR08" H 4150 2800 50  0001 C CNN
-F 1 "+9V" V 4165 3078 50  0000 L CNN
-F 2 "" H 4150 2950 50  0001 C CNN
-F 3 "" H 4150 2950 50  0001 C CNN
-	1    4150 2950
-	0    1    1    0
-$EndComp
-$Comp
-L power:GND #PWR06
-U 1 1 00000000
-P 1750 3100
-F 0 "#PWR06" H 1750 2850 50  0001 C CNN
-F 1 "GND" H 1755 2927 50  0000 C CNN
-F 2 "" H 1750 3100 50  0001 C CNN
-F 3 "" H 1750 3100 50  0001 C CNN
-	1    1750 3100
+L power:+9V #PWR06
+U 1 1 5E802FD9
+P 1950 2700
+F 0 "#PWR06" H 1950 2550 50  0001 C CNN
+F 1 "+9V" H 1850 2803 50  0000 C CNN
+F 2 "" H 1950 2700 50  0001 C CNN
+F 3 "" H 1950 2700 50  0001 C CNN
+	1    1950 2700
+	1    0    0    -1
+$EndComp
+$Comp
+L power:+9V #PWR0102
+U 1 1 5E75D081
+P 3750 2950
+F 0 "#PWR0102" H 3750 2800 50  0001 C CNN
+F 1 "+9V" H 3765 3123 50  0000 C CNN
+F 2 "" H 3750 2950 50  0001 C CNN
+F 3 "" H 3750 2950 50  0001 C CNN
+	1    3750 2950
+	1    0    0    -1
+$EndComp
+$Comp
+L power:+9V #PWR07
+U 1 1 5E830921
+P 3900 3500
+F 0 "#PWR07" H 3900 3350 50  0001 C CNN
+F 1 "+9V" H 3915 3327 50  0000 C CNN
+F 2 "" H 3900 3500 50  0001 C CNN
+F 3 "" H 3900 3500 50  0001 C CNN
+	1    3900 3500
+	1    0    0    -1
+$EndComp
+$Comp
+L power:GND #PWR0101
+U 1 1 5E75D08D
+P 2050 3100
+F 0 "#PWR0101" H 2050 2850 50  0001 C CNN
+F 1 "GND" H 2055 2927 50  0000 C CNN
+F 2 "" H 2050 3100 50  0001 C CNN
+F 3 "" H 2050 3100 50  0001 C CNN
+	1    2050 3100
 	1    0    0    -1
 $EndComp
 $Comp
 L power:GND #PWR02
-U 1 1 00000000
+U 1 1 5E75D099
 P 2350 2450
 F 0 "#PWR02" H 2350 2200 50  0001 C CNN
@@
 $Comp
 L power:GND #PWR03
-U 1 1 00000000
+U 1 1 5E75D0A5
 P 2950 2450
 F 0 "#PWR03" H 2950 2200 50  0001 C CNN
@@
 $EndComp
 $Comp
-L power:GND #PWR07
-U 1 1 00000000
-P 3150 3100
-F 0 "#PWR07" H 3150 2850 50  0001 C CNN
-F 1 "GND" H 3155 2927 50  0000 C CNN
-F 2 "" H 3150 3100 50  0001 C CNN
-F 3 "" H 3150 3100 50  0001 C CNN
-	1    3150 3100
-	1    0    0    -1
-$EndComp
-$Comp
 L power:GND #PWR04
-U 1 1 00000000
+U 1 1 5E75D0B1
 P 3600 2450
 F 0 "#PWR04" H 3600 2200 50  0001 C CNN
@@
 $EndComp
 $Comp
-L power:GND #PWR09
-U 1 1 00000000
-P 4150 3150
-F 0 "#PWR09" H 4150 2900 50  0001 C CNN
-F 1 "GND" H 4155 2977 50  0000 C CNN
-F 2 "" H 4150 3150 50  0001 C CNN
-F 3 "" H 4150 3150 50  0001 C CNN
-	1    4150 3150
+L power:GND #PWR0103
+U 1 1 5E75D0BD
+P 3750 3050
+F 0 "#PWR0103" H 3750 2800 50  0001 C CNN
+F 1 "GND" H 3755 2877 50  0000 C CNN
+F 2 "" H 3750 3050 50  0001 C CNN
+F 3 "" H 3750 3050 50  0001 C CNN
+	1    3750 3050
 	1    0    0    -1
 $EndComp
 $Comp
 L power:GND #PWR05
-U 1 1 00000000
+U 1 1 5E75D0C9
 P 4300 2450
 F 0 "#PWR05" H 4300 2200 50  0001 C CNN
@@
 $EndComp
 $Comp
+L power:GND #PWR?
+U 1 1 5E83E43D
+P 4500 3750
+F 0 "#PWR?" H 4500 3500 50  0001 C CNN
+F 1 "GND" H 4505 3923 50  0000 C CNN
+F 2 "" H 4500 3750 50  0001 C CNN
+F 3 "" H 4500 3750 50  0001 C CNN
+	1    4500 3750
+	1    0    0    -1
+$EndComp
+$Comp
+L Device:R R5
+U 1 1 5E802098
+P 1800 2850
+F 0 "R5" V 1894 2844 50  0000 C CNN
+F 1 "4k7" V 1685 2835 50  0000 C CNN
+F 2 "resistors:0.3%22.B" V 1730 2850 50  0001 C CNN
+F 3 "~" H 1800 2850 50  0001 C CNN
+	1    1800 2850
+	0    -1   -1   0
+$EndComp
+$Comp
 L Device:R R2
-U 1 1 00000000
+U 1 1 5E75D0D5
 P 2950 1600
 F 0 "R2" H 3020 1645 50  0000 L CNN
@@
 $Comp
 L Device:R R1
-U 1 1 00000000
+U 1 1 5E75D0E1
 P 2950 2150
 F 0 "R1" H 3020 2195 50  0000 L CNN
@@
 $Comp
 L Device:R R3
-U 1 1 00000000
+U 1 1 5E75D0ED
 P 3600 1100
 F 0 "R3" H 3670 1145 50  0000 L CNN
@@
 $Comp
 L Device:R R4
-U 1 1 00000000
+U 1 1 5E75D0F9
 P 4300 2150
 F 0 "R4" H 4370 2195 50  0000 L CNN
@@
 $EndComp
 $Comp
+L Connector_Generic:Conn_01x01 J3
+U 1 1 5E82F8EF
+P 4100 3500
+F 0 "J3" H 4180 3458 50  0000 L CNN
+F 1 "Conn_01x01" H 4180 3549 50  0000 L CNN
+F 2 "rockola_kicad_footprints:V+_TOP_TEXT" H 4100 3500 50  0001 C CNN
+F 3 "~" H 4100 3500 50  0001 C CNN
+	1    4100 3500
+	1    0    0    -1
+$EndComp
+$Comp
+L Connector_Generic:Conn_01x01 J4
+U 1 1 5E8362AC
+P 4700 3750
+F 0 "J4" H 4780 3708 50  0000 L CNN
+F 1 "Conn_01x01" H 4780 3799 50  0000 L CNN
+F 2 "supply_pins:PAD1" H 4700 3750 50  0001 C CNN
+F 3 "~" H 4700 3750 50  0001 C CNN
+	1    4700 3750
+	1    0    0    -1
+$EndComp
+$Comp
 L Device:D D1
-U 1 1 00000000
+U 1 1 5E75D105
 P 2350 1600
 F 0 "D1" V 2305 1679 50  0000 L CNN
@@
 $Comp
 L Device:D D2
-U 1 1 00000000
+U 1 1 5E75D111
 P 2350 2150
 F 0 "D2" V 2305 2229 50  0000 L CNN
@@
 $EndComp
 $Comp
+L Device:LED D3
+U 1 1 5E800FFD
+P 1450 2850
+F 0 "D3" H 1443 2634 50  0000 C CNN
+F 1 "LED" H 1443 2725 50  0000 C CNN
+F 2 "LED_THT:LED_D3.0mm" H 1450 2850 50  0001 C CNN
+F 3 "~" H 1450 2850 50  0001 C CNN
+	1    1450 2850
+	1    0    0    -1
+$EndComp
+$Comp
+L Connector_Generic:Conn_01x02 J2
+U 1 1 5E75D11D
+P 4100 2950
+F 0 "J2" H 4180 2942 50  0000 L CNN
+F 1 "Conn_01x02" H 4180 2851 50  0000 L CNN
+F 2 "rockola_kicad_footprints:Power_Header_2pin_VERTICAL" H 4100 2950 50  0001 C CNN
+F 3 "~" H 4100 2950 50  0001 C CNN
+	1    4100 2950
+	1    0    0    -1
+$EndComp
+$Comp
 L Device:C C1
-U 1 1 00000000
+U 1 1 5E75D129
 P 1950 1850
 F 0 "C1" V 2201 1850 50  0000 C CNN
@@
 $Comp
 L Device:CP C2
-U 1 1 00000000
+U 1 1 5E75D135
 P 4150 1450
 F 0 "C2" V 4404 1450 50  0000 C CNN
@@
 $Comp
 L Device:R_POT RV1
-U 1 1 00000000
+U 1 1 5E75D141
 P 3600 2150
 F 0 "RV1" H 3530 2105 50  0000 R CNN
 F 1 "C5k" H 3530 2195 50  0000 R CNN
-F 2 "potentiometers:16MM_C.MOUNT" H 3600 2150 50  0001 C CNN
+F 2 "rockola_kicad_footprints:16mm_BoardMount" H 3600 2150 50  0001 C CNN
 F 3 "~" H 3600 2150 50  0001 C CNN
 	1    3600 2150
@@
 $EndComp
 $Comp
-L Connector:AudioJack2 J1
-U 1 1 00000000
-P 1200 3100
-F 0 "J1" H 1232 3423 50  0000 C CNN
-F 1 "Input" H 1232 3332 50  0000 C CNN
-F 2 "jacks:2PADS_TS" H 1200 3100 50  0001 C CNN
-F 3 "~" H 1200 3100 50  0001 C CNN
-	1    1200 3100
-	1    0    0    -1
-$EndComp
-$Comp
-L Connector:AudioJack2 J2
-U 1 1 00000000
-P 2500 3100
-F 0 "J2" H 2532 3423 50  0000 C CNN
-F 1 "Output" H 2532 3332 50  0000 C CNN
-F 2 "jacks:2PADS_TS" H 2500 3100 50  0001 C CNN
-F 3 "~" H 2500 3100 50  0001 C CNN
-	1    2500 3100
-	1    0    0    -1
-$EndComp
-$Comp
-L Connector:Barrel_Jack J3
-U 1 1 00000000
-P 3750 3050
-F 0 "J3" H 3520 3008 50  0000 R CNN
-F 1 "Power" H 3520 3099 50  0000 R CNN
-F 2 "jacks:DC_TS" H 3800 3010 50  0001 C CNN
-F 3 "~" H 3800 3010 50  0001 C CNN
-	1    3750 3050
-	1    0    0    1
+L rockola_kicad_symbols:Stomp_Connector J1
+U 1 1 5E7ED44E
+P 2700 3000
+F 0 "J1" H 2780 3008 50  0000 L CNN
+F 1 "Stomp_Connector" H 2780 3099 50  0000 L CNN
+F 2 "rockola_kicad_footprints:Stomp_4pin" H 2700 3000 50  0001 C CNN
+F 3 "~" H 2700 3000 50  0001 C CNN
+	1    2700 3000
+	1    0    0    -1
 $EndComp
 $Comp
 L Transistor_FET:BS170 Q1
-U 1 1 00000000
+U 1 1 5E75D159
 P 3500 1650
 F 0 "Q1" H 3705 1695 50  0000 L CNN
 F 1 "BS170" H 3705 1605 50  0000 L CNN
-F 2 "transistors-BJT:TO92" H 3700 1575 50  0001 L CIN
+F 2 "rockola_kicad_footprints:TO92_DGS" H 3700 1575 50  0001 L CIN
 F 3 "http://www.fairchildsemi.com/ds/BS/BS170.pdf" H 3500 1650 50  0001 L CNN
 	1    3500 1650

Commit message: v0.2: Superheated SHO
Parts:
- added C3: 100n, rockola_kicad_footprints:C_Box_7.2_2.5, symbol Device:C
- added C4: 10u, caps-elec:0502, symbol Device:CP
- added D4: 9V1, diodes:DO41-3, symbol Device:D_Zener
- added Q2: MMBF5457, rockola_kicad_footprints:SOT-23_NJFET_DSG, symbol rockola_kicad_symbols:MMBF5457
- added R6, R7: 1M, resistors:0.3%22.B, symbol Device:R
- added SW1: SW_SPDT, switches:SPDT.WIRE, symbol Switch:SW_SPDT
- C1: footprint caps-film:0.2_22.MED -> rockola_kicad_footprints:C_Box_7.2_2.5
- D1, D2: footprint diodes:DO35-2 -> diodes:DO35-3
- J1: footprint rockola_kicad_footprints:Stomp_4pin -> rockola_kicad_footprints:Stomp_4pin_ALT2
- R3: value 5k1 -> 4k7
- RV1: value C5k -> B1k
Connections:
- net +9V: now also Q2.D, R6.1
- net GND: now also C4.2, R7.2; no longer RV1.2
- net at C2.1, Q1.1 (D), R2.1: now also SW1.2 (B); no longer R3.2
- net at C1.2, D1.2 (A), D2.1 (K)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: now also D4.1 (K)
- net at Q1.3 (S), RV1.3: now also D4.2 (A)
- new net: R3.2, SW1.1 (A)
- new net: C4.1, RV1.2
- new net: C3.2, Q2.S, SW1.3 (C)
- new net: C3.1, Q2.G, R6.2, R7.1
Other:
- note added: "2020-04-02"
- note added: "Basic SHO:\nRV1 = C5k\nR3 = 5k1\nJumper C4, SW1 (1-2)\nOmit R6, R7, C3, Q2\nOptional (not recommended):\nOmit D1, D2, D4"
- note added: "Hot"
- note added: "SHO and Superheated SHO"
- note added: "Superduro"
- note added: "Superheated"
- note added: "v0.2"
- moved on the sheet: C1, C2, D1, D2, D3, J1, J2, J3, J4, Q1, R1, R2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
